File: For Micro/control-module.kicad_pcb (KiCad board)
At the start: 2 copper layers, 59.7 x 66 mm, 37 parts, among them J1 For Expansion, J2 For Light Sensor, J3 From Solar Panel, J4 To Flow Module (F), J5 For Flow Module b, J6 For Flow Module a, Q1 NMOS, Q2 NMOS, Q3 NMOS, Q4 NMOS, U1 TR_SERIES, U2 TR_SERIES, U3 ARDUINO_MICRO_SHIELD

Commit message: Final CAD for Micro
Parts:
- added REF**: MountingHole_2.2mm_M2, Mounting_Holes:MountingHole_2.2mm_M2, F.Cu at (134.6, 100.8)
- added REF**: MountingHole_2.2mm_M2, Mounting_Holes:MountingHole_2.2mm_M2, F.Cu at (86.4, 98.0)
- added REF**: MountingHole_2.2mm_M2, Mounting_Holes:MountingHole_2.2mm_M2, F.Cu at (86.4, 151.1)
Routing:
- net GND: track 0.00 -> 184.2 mm, vias 0 -> 17
- net VCC+5V: track 0.00 -> 157.6 mm, vias 0 -> 7
- net SDAC: track 0.00 -> 84.9 mm
- net 5V: track 8.22 -> 92.1 mm
- net INPUT2: track 0.00 -> 81.4 mm, vias 0 -> 6
- net SCLC: track 0.00 -> 80.2 mm
- net Net-(C4-Pad1): track 50.3 -> 128.7 mm, vias 2 -> 6
- net EN2: track 0.00 -> 74.8 mm, vias 0 -> 2
- net INPUT5: track 0.00 -> 71.9 mm
- net VCC+EXP: track 0.00 -> 70.5 mm, vias 0 -> 2
- net INPUT4: track 0.00 -> 63.4 mm, vias 0 -> 5
- net EN1: track 0.00 -> 57.3 mm, vias 0 -> 4
- net VCC+LS: track 0.00 -> 56.7 mm, vias 0 -> 2
- net SDAB: track 0.00 -> 53.5 mm, vias 0 -> 2
- net INPUT3: track 0.00 -> 50.2 mm, vias 0 -> 3
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- added copper zone on B.Cu, net GND
- added copper zone on F.Cu, net GND
Other:
- board size 59.7 x 66 mm -> 63.5 x 68.1 mm
